Commit message: lidar working on rviz, not localized yet though

File: occupancy_map/simple_robot.urdf (robot description, URDF)
Before this commit: robot simple_ball, 1 links, 0 joints
Links:
- added link laser_frame; visual cylinder length=0.04 radius=0.05
Joints:
- added joint laser_joint: type fixed, parent base_link, child laser_frame, origin xyz=0 0 0.2 rpy=0 0 0

Commit message: Update README.md file

File: occupancy_map/simple_robot.urdf (robot description, URDF)
Before this commit: robot simple_ball, 2 links, 1 joints
Links:
- removed link base_link
- removed link laser_frame
- added link wizard/base_link; visual box size=0.1 0.05 0.05; visual sphere radius=0.3
Joints:
- removed joint laser_joint
